Commit message: Changed downsample parameter from 1 to 10, RT factor jumped from 0.4 to 0.99.

File: husky_with_livox/urdf/livox_mid70.xacro (robot description, xacro)
@@ -8,5 +8,5 @@
   <xacro:property name="ros_topic" value="scan"/>
   <xacro:property name="samples" value="10000"/>
-  <xacro:property name="downsample" value="1"/>
+  <xacro:property name="downsample" value="10"/>
   <xacro:macro name="null_inertial">
     <inertial>

Commit message: Added customized xacro to be copied to livox_laser_simulation.

File: husky_with_livox/urdf/livox_mid70.xacro (robot description, xacro)
@@ -17,4 +17,6 @@
     </inertial>
   </xacro:macro>
+  <!-- 10Hz seems to be normal publish rate for Solid-state Lidars -->
+  <!-- https://www.mdpi.com/1424-8220/21/5/1773/htm-->
   <xacro:macro name="Livox_Mid_gazebo_sensor" params="visualize:=True update_rate:=10 resolution:=0.002 noise_mean:=0.0 noise_stddev:=0.01 name:=livox">
     <gazebo reference="${name}">
@@ -66,4 +68,7 @@
         <origin xyz="0.00 0 0.00" rpy="0 0 0"/>
         <geometry>
+          <!-- Tried to add custom converted .stp mid70 mesh to the simu. env. but didn't work well -->
+          <!-- Simulation physics were buggy. -->
+          <!-- <mesh filename="$(find husky_with_livox)/meshes/livox_mid70.dae"> -->
           <mesh filename="package://livox_laser_simulation/meshes/livox_mid40.dae">
           </mesh>
@@ -73,4 +78,5 @@
           <origin xyz="0 0 0" rpy="0 0 0" />
           <geometry>
+          <!-- <mesh filename="$(find husky_with_livox)/meshes/livox_mid70.dae"> -->
           <mesh filename="package://livox_laser_simulation/meshes/livox_mid40.dae">
           </mesh>

Commit message: Changed downsample to 1 so that we get 10k points per message and downsample it in the pre-processing stage.

File: husky_with_livox/urdf/livox_mid70.xacro (robot description, xacro)
@@ -8,5 +8,6 @@
   <xacro:property name="ros_topic" value="scan"/>
   <xacro:property name="samples" value="10000"/>
-  <xacro:property name="downsample" value="10"/>
+  <!-- Kept downsample to 1 so that we get 10k points per message. -->
+  <xacro:property name="downsample" value="1"/>
   <xacro:macro name="null_inertial">
     <inertial>
