Commit message: Fixed husky to livox URDF.

File: husky_with_livox/urdf/custom_description.urdf.xacro (robot description, xacro)
@@ -328,22 +328,13 @@
   <!-- Optional for Clearpath internal softwares -->
   <xacro:include filename="$(arg cpr_urdf_extras)" />
-  <!-- Test to see a customization inside the original package works -->
-  <link name="bowler_link">
-    <visual>
-      <geometry>
-        <mesh filename="package://husky_custom_description/meshes/red_bowler.dae" />
-      </geometry>
-    </visual>
-    <collision>
-      <origin xyz="0 0 0.07" rpy="0 0 0" />
-      <geometry>
-        <box size="0.32 0.25 0.14" rpy="0 0 0"/>
-      </geometry>
-    </collision>
-  </link>
-  <joint name="bowler_joint" type="fixed">
+  <!-- Livox Sensor -->
+  <xacro:include filename="$(find livox_laser_simulation)/urdf/livox_mid70.xacro" />
+  <xacro:property name="livox_lidar" value="livoxx"/>
+  <!-- Instantiating the xacro macro within livox_mid70.xacro -->
+  <xacro:Livox_Mid70 name="${livox_lidar}"/>
+  <joint name="husky_to_livox_joint" type="fixed">
     <parent link="top_plate_link" />
-    <child link="bowler_link" />
-    <origin xyz="0.1 -0.1 0" rpy="0 0 0.5" />
+    <child link="${livox_lidar}_base" />
+    <origin xyz="0 0 0" rpy="0 0 0" />
   </joint>
 </robot>

Commit message: Adjusted livox position wrt. to husky.

File: husky_with_livox/urdf/custom_description.urdf.xacro (robot description, xacro)
@@ -336,5 +336,5 @@
     <parent link="top_plate_link" />
     <child link="${livox_lidar}_base" />
-    <origin xyz="0 0 0" rpy="0 0 0" />
+    <origin xyz="0.36 0 0.015" rpy="0 0 0" />
   </joint>
 </robot>

Commit message: Adjusted Z position of Livox, was way too low.

File: husky_with_livox/urdf/custom_description.urdf.xacro (robot description, xacro)
@@ -336,5 +336,5 @@
     <parent link="top_plate_link" />
     <child link="${livox_lidar}_base" />
-    <origin xyz="0.36 0 0.015" rpy="0 0 0" />
+    <origin xyz="0.34 0 0.045" rpy="0 0 0" />
   </joint>
 </robot>

Commit message: Adjusted frame_id name to livox so that RViz detects the correct frame_id when publishing the PointCloud data. Working.

File: husky_with_livox/urdf/custom_description.urdf.xacro (robot description, xacro)
@@ -330,5 +330,5 @@
   <!-- Livox Sensor -->
   <xacro:include filename="$(find livox_laser_simulation)/urdf/livox_mid70.xacro" />
-  <xacro:property name="livox_lidar" value="livoxx"/>
+  <xacro:property name="livox_lidar" value="livox"/>
   <!-- Instantiating the xacro macro within livox_mid70.xacro -->
   <xacro:Livox_Mid70 name="${livox_lidar}"/>
